File: hardware/goodpocketwatch31/usb.sch (KiCad schematic (older format))
At the start: 9 parts, among them J2 DX07S016JA1R1500, U4 SN74AXC4T774RSVR, U5 FT232RQ-REEL

Commit message: Bit more drafting, almost done with the pocket watch. #147
Parts:
- added C11, C12, C13: 0.1uF, Capacitor_SMD:C_0402_1005Metric, symbol Device:C
Connections:
- wire segments 47 -> 53
Changed lines of the file:
@@
 NoConn ~ 8300 2050
 NoConn ~ 8300 1450
+$Comp
+L Device:C C11
+U 1 1 5FF05C3F
+P 2700 4750
+F 0 "C11" H 2815 4796 50  0000 L CNN
+F 1 "0.1uF" H 2750 4650 50  0000 L CNN
+F 2 "Capacitor_SMD:C_0402_1005Metric" H 2738 4600 50  0001 C CNN
+F 3 "~" H 2700 4750 50  0001 C CNN
+	1    2700 4750
+	1    0    0    -1
+$EndComp
+$Comp
+L Device:C C12
+U 1 1 5FF062B5
+P 3100 4750
+F 0 "C12" H 3215 4796 50  0000 L CNN
+F 1 "0.1uF" H 3150 4650 50  0000 L CNN
+F 2 "Capacitor_SMD:C_0402_1005Metric" H 3138 4600 50  0001 C CNN
+F 3 "~" H 3100 4750 50  0001 C CNN
+	1    3100 4750
+	1    0    0    -1
+$EndComp
+$Comp
+L Device:C C13
+U 1 1 5FF06586
+P 3450 4750
+F 0 "C13" H 3565 4796 50  0000 L CNN
+F 1 "0.1uF" H 3500 4650 50  0000 L CNN
+F 2 "Capacitor_SMD:C_0402_1005Metric" H 3488 4600 50  0001 C CNN
+F 3 "~" H 3450 4750 50  0001 C CNN
+	1    3450 4750
+	1    0    0    -1
+$EndComp
+$Comp
+L power:GND #PWR020
+U 1 1 5FF09A74
+P 2700 5000
+F 0 "#PWR020" H 2700 4750 50  0001 C CNN
+F 1 "GND" H 2705 4827 50  0000 C CNN
+F 2 "" H 2700 5000 50  0001 C CNN
+F 3 "" H 2700 5000 50  0001 C CNN
+	1    2700 5000
+	1    0    0    -1
+$EndComp
+$Comp
+L power:GND #PWR021
+U 1 1 5FF0A1FE
+P 3100 5000
+F 0 "#PWR021" H 3100 4750 50  0001 C CNN
+F 1 "GND" H 3105 4827 50  0000 C CNN
+F 2 "" H 3100 5000 50  0001 C CNN
+F 3 "" H 3100 5000 50  0001 C CNN
+	1    3100 5000
+	1    0    0    -1
+$EndComp
+$Comp
+L power:GND #PWR022
+U 1 1 5FF0A398
+P 3450 5000
+F 0 "#PWR022" H 3450 4750 50  0001 C CNN
+F 1 "GND" H 3455 4827 50  0000 C CNN
+F 2 "" H 3450 5000 50  0001 C CNN
+F 3 "" H 3450 5000 50  0001 C CNN
+	1    3450 5000
+	1    0    0    -1
+$EndComp
+Wire Wire Line
+	2700 4900 2700 5000
+Wire Wire Line
+	3100 4900 3100 5000
+Wire Wire Line
+	3450 4900 3450 5000
+Wire Wire Line
+	2700 4600 2700 4400
+Wire Wire Line
+	3100 4600 3100 4400
+Wire Wire Line
+	3450 4600 3450 4400
+Text Label 2700 4600 1    60   ~ 0
+VCC
+Text Label 3100 4600 1    60   ~ 0
+VCCB
+Text Label 3450 4600 1    60   ~ 0
+VBUS
 $EndSCHEMATC
