File: hardware/goodpocketwatch31/keypad.sch (KiCad schematic (older format))
At the start: 16 parts, among them SW0 SW_Push, SW1 SW_Push, SW10 SW_Push, SW11 SW_Push, SW12 SW_Push, SW13 SW_Push, SW14 SW_Push, SW15 SW_Push, SW2 SW_Push, SW3 SW_Push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

Commit message: Layou of GPW31 is complete except for the SMA connector. #147
Parts:
- added SW16, SW17: SW_Push, goodpocketwatch31:TL6700, symbol Switch:SW_Push
Connections:
- net labels added: GND, MODE, PRGM
- wire segments 48 -> 52
Changed lines of the file:
@@
 Text GLabel 6500 2000 1    60   Input ~ 0
 P17
+Text GLabel 7950 2800 0    60   Input ~ 0
+MODE
+Text GLabel 7950 3250 0    60   Input ~ 0
+PRGM
+$Comp
+L Switch:SW_Push SW16
+U 1 1 5FE94086
+P 8300 2800
+F 0 "SW16" H 8300 3085 50  0000 C CNN
+F 1 "SW_Push" H 8300 2994 50  0000 C CNN
+F 2 "goodpocketwatch31:TL6700" H 8300 3000 50  0001 C CNN
+F 3 "~" H 8300 3000 50  0001 C CNN
+	1    8300 2800
+	1    0    0    -1
+$EndComp
+$Comp
+L Switch:SW_Push SW17
+U 1 1 5FE94597
+P 8300 3250
+F 0 "SW17" H 8300 3535 50  0000 C CNN
+F 1 "SW_Push" H 8300 3444 50  0000 C CNN
+F 2 "goodpocketwatch31:TL6700" H 8300 3450 50  0001 C CNN
+F 3 "~" H 8300 3450 50  0001 C CNN
+	1    8300 3250
+	1    0    0    -1
+$EndComp
+Wire Wire Line
+	7950 2800 8100 2800
+Wire Wire Line
+	7950 3250 8100 3250
+Wire Wire Line
+	8500 2800 8750 2800
+Wire Wire Line
+	8500 3250 8750 3250
+Text Label 8550 2800 0    60   ~ 0
+GND
+Text Label 8550 3250 0    60   ~ 0
+GND
 $EndSCHEMATC
