File: hardware/goodpocketwatch31/goodpocketwatch31.kicad_pcb (KiCad board)
At the start: 2 copper layers, 75.2 x 101.2 mm, 47 parts, among them J1 ANT_U.FL, J2 DX07S016JA1R1500, SW0 SW_Push, SW1 SW_Push, SW10 SW_Push, SW11 SW_Push, SW12 SW_Push, SW13 SW_Push, SW14 SW_Push, SW15 SW_Push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

Commit message: Most of the layout, but still needs some caps. #147
Parts:
- added BZ1: Buzzer, goodpocketwatch31:PT-1203-3, F.Cu at (78.6, 79.9)
- U4: value SN74AXC4T774RSVR -> SN74AXC4T774
- U5: value FT232RQ-REEL -> FT232RQ
- moved D1 22.2 mm to (130.1, 80.9), turned to 180 degrees
- moved R5 22.2 mm to (133.1, 80.9), turned to 180 degrees
- moved D2 21.3 mm to (130.1, 83.9), turned to 180 degrees
- moved R6 21.2 mm to (133.1, 83.9), turned to 180 degrees
- moved R3 15.1 mm to (145.6, 74.9), turned to 270 degrees
- moved U4 12.5 mm to (142.4, 90.6), turned to 90 degrees
- moved J2 3.00 mm to (138.6, 76.4)
- moved R4 2.42 mm to (131.6, 74.9), turned to 90 degrees
- moved U5 2.00 mm to (140.6, 84.4), turned to 180 degrees
Connections:
- C8 pad 2: Net-(C8-Pad2) -> GND
- C9 pad 2: Net-(C9-Pad2) -> GND
- D1 pad 2: VCC -> /USB/VBUS
- D2 pad 2: VCC -> /USB/VBUS
Routing:
- net P20: track 4.09 -> 135.6 mm
- net P26: track 5.70 -> 122.2 mm, vias 0 -> 2
- net P21: track 3.39 -> 113.9 mm, vias 0 -> 2
- net P25: track 4.02 -> 105.2 mm, vias 0 -> 2
- net P17: track 5.18 -> 94.3 mm
- net P22: track 2.51 -> 89.9 mm, vias 0 -> 2
- net P24: track 3.23 -> 88.0 mm, vias 0 -> 2
- net P23: track 3.25 -> 71.1 mm
- net GND: track 15.7 -> 48.6 mm, vias 49 -> 52
- net /USB/VBUS: track 0.00 -> 23.9 mm
- net /USB/VCCB: track 0.00 -> 21.0 mm, vias 0 -> 3
- net Net-(J2-Pad9): track 0.00 -> 9.66 mm, vias 0 -> 2
- net /USB/USBDM: track 0.00 -> 9.18 mm
- net Net-(J2-Pad3): track 0.00 -> 7.76 mm
- net /USB/USBDP: track 0.00 -> 7.68 mm
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
Commit message: Bit more drafting, almost done with the pocket watch. #147
Parts:
- added BT1: AAAA, goodpocketwatch31:BE-AAAA-PC, B.Cu at (78.0, 122.0)
- added BT2: AAAA, goodpocketwatch31:BE-AAAA-PC, B.Cu at (139.6, 122.0)
- added C11: 0.1uF, Capacitor_SMD:C_0402_1005Metric, F.Cu at (138.6, 89.4)
- added C12: 0.1uF, Capacitor_SMD:C_0402_1005Metric, F.Cu at (137.6, 80.4)
- added C13: 0.1uF, Capacitor_SMD:C_0402_1005Metric, F.Cu at (136.6, 82.9)
- moved BZ1 2.12 mm to (80.1, 81.4)
Routing:
- net GND: track 48.6 -> 54.1 mm
- net VCC: track 61.4 -> 64.6 mm
- net /USB/RXLED: track 6.31 -> 7.57 mm
- net /USB/VCCB: track 21.0 -> 22.0 mm
- net /USB/VBUS: track 23.9 -> 24.5 mm

Commit message: Layou of GPW31 is complete except for the SMA connector. #147
Parts:
- added SW16: SW_Push, goodpocketwatch31:TL6700, F.Cu at (82.6, 85.4)
- added SW17: SW_Push, goodpocketwatch31:TL6700, B.Cu at (124.1, 115.9)
- BZ1: moved to B.Cu
- U4: value SN74AXC4T774 -> SN74AXC4T77
- U5: value FT232RQ -> FT232RQ-REEL
- moved BT1 62.0 mm to (140.0, 122.0)
- moved BT2 61.6 mm to (78.0, 122.0)
- moved BZ1 42.4 mm to (109.1, 112.4), turned to 270 degrees
Routing:
- net GND: track 54.1 -> 183.6 mm, vias 52 -> 57
- net Net-(BT1-Pad2): track 0.00 -> 106.9 mm, vias 0 -> 2
- net MODE: track 17.4 -> 92.1 mm, vias 0 -> 2
- net PRGM: track 11.6 -> 83.6 mm, vias 0 -> 2
- net VCC: track 64.6 -> 134.2 mm, vias 4 -> 7
- net TST: track 6.30 -> 52.5 mm, vias 0 -> 2
- net RST: track 12.5 -> 57.7 mm, vias 1 -> 3
- net /BUZZ: track 10.1 -> 42.8 mm, vias 1 -> 2
- net P17: track 94.3 -> 98.6 mm
- net /USB/VCCB: track 22.0 -> 18.6 mm
- net P20: track 135.6 -> 136.8 mm
Other:
- board text added: "MODE"
- board text added: "RX"
- board text added: "TX"

Commit message: Adds an edge-mount SMA connector, handy for RF accessories. #147
Parts:
- added J3: SMA, Connector_Coaxial:SMA_Amphenol_132289_EdgeMount, F.Cu at (85.6, 75.4)
- U4: value SN74AXC4T77 -> SN74AXC4T774RSVR
Routing:
- net Net-(A1-Pad1): track 28.3 -> 44.0 mm
- net GND: track 183.6 -> 190.6 mm, vias 57 -> 68
